File: I2C-23017.sch (EAGLE design)
At the start: 4 parts

Commit message: new IOB and power connectors
Parts:
- added C1, C3: 0.1uF, SPCoast:CAP0805
- added C2: 10uF, SPCoast:CAP0805
- added C4: 220uF, SPCoast:CAP-POL0810
- added CON1, CON2: (no value), SPCoast:CONNECTOR-I2CLEFT
- added IC1: MCP23017SO, microchip:MCP23017SO
- added LED1, LED10, LED11, LED12, LED13, LED14, LED15, LED16, LED2, LED3, LED4, LED5, LED6, LED7, LED8, LED9: Y, SPCoast:LED0603-LED
- added LED18: GREEN, SPCoast:LED0603-LED
- added POWER: 9-12Vdc, SPCoast:DOC-POWER_LABEL
- added Q0, Q1, Q10, Q11, Q12, Q13, Q14, Q15, Q2, Q3, Q4, Q5, Q6, Q7, Q8, Q9: P-FET, SPCoast:MOSFET-P-044021001
- added R1, R2, R3: 10K, SPCoast:R0603-RES
- added R10, R11, R12, R13, R14, R15, R16, R17, R21, R22, R4, R5, R6, R7, R8, R9: 2K0, SPCoast:R0805-RES
- added R18: 2K2, SPCoast:R0603-RES
- added R19, R20: 4k7, SPCoast:R0603-RES
- added SCL: SCL, SPCoast:JUMPER-2PTH_LOCK
- added SDA: SDA, SPCoast:JUMPER-2PTH_LOCK
- added SW1: (no value), SPCoast:SW_DIP-4
- added U$1, U$2, U$3, U$4: CONNECTOR-IO4-IOBBARE, SPCoast:CONNECTOR-IO4-IOBBARE
- added VIN: (no value), SPCoast:CONNECTOR-DC-POWER-RA
- added VIN1: CONNECTOR-POWER-R, SPCoast:CONNECTOR-POWER-R
- added VIN2: CONNECTOR-POWER-L, SPCoast:CONNECTOR-POWER-L
- added VR1: CJ7805, SPCoast:VREG-DPAK-5
- BOARD1: value BOARD80X100 -> BOARD80X100-IOB; device SPCoast:BOARD80X100 -> SPCoast:BOARD80X100-IOB
Connections:
- new net +9V: C1.1, U$1.VIN, U$2.VIN, U$3.VIN, U$4.VIN, VIN.1, VIN1.V+, VIN2.V+, VR1.IN
- new net A0: IC1.A0, R1.1, SW1.8
- new net A1: IC1.A1, R2.1, SW1.7
- new net A3: IC1.A2, R3.1, SW1.6
- new net GND: C1.2, C2.2, C3.2, C4.-, CON1.GND, CON2.GND, IC1.VSS, LED1.C, LED10.C, LED11.C, LED12.C, LED13.C, LED14.C, LED15.C, LED16.C, LED2.C, LED3.C, LED4.C, LED5.C, LED6.C, LED7.C, LED8.C, LED9.C, R18.2, SW1.1, SW1.2, SW1.3, U$1.GND, U$2.GND, U$3.GND, U$4.GND, VIN.2, VIN.3, VIN1.GND, VIN2.GND, VR1.GND
- new net N$1: Q4.D, R11.2
- new net N$10: Q8.D, R15.2
- new net N$11: Q9.D, R12.2
- new net N$12: Q10.D, R13.2
- new net N$13: Q11.D, R14.2
- new net N$14: LED12.A, R15.1
- new net N$15: LED9.A, R12.1
- new net N$2: CON1.V+, CON2.V+
- new net N$20: R20.1, SCL.1
- new net N$21: R19.1, SDA.1
- new net N$22: LED18.C, R18.1
- new net N$23: LED10.A, R13.1
- new net N$24: LED11.A, R14.1
- new net N$28: Q12.D, R22.2
- new net N$29: Q13.D, R16.2
- new net N$3: Q5.D, R8.2
- new net N$30: Q14.D, R17.2
- new net N$31: Q15.D, R21.2
- new net N$32: LED16.A, R22.1
- new net N$33: LED13.A, R16.1
- new net N$34: LED14.A, R17.1
- new net N$35: LED15.A, R21.1
- new net N$4: Q6.D, R9.2
- new net N$44: Q0.D, R7.2
- new net N$45: Q1.D, R4.2
- new net N$46: Q2.D, R5.2
- new net N$47: Q3.D, R6.2
- new net N$48: LED1.A, R7.1
- new net N$49: LED2.A, R4.1
- new net N$5: Q7.D, R10.2
- new net N$50: LED3.A, R5.1
- new net N$51: LED4.A, R6.1
- new net N$6: LED8.A, R11.1
- new net N$7: LED5.A, R8.1
- new net N$8: LED6.A, R9.1
- new net N$9: LED7.A, R10.1
- new net P1: IC1.GPA0, Q0.G, U$1.P1
- new net P10: IC1.GPB1, Q9.G, U$3.P2
- new net P11: IC1.GPB2, Q10.G, U$3.P3
- new net P12: IC1.GPB3, Q11.G, U$3.P4
- new net P13: IC1.GPB4, Q12.G, U$4.P1
- new net P14: IC1.GPB5, Q13.G, U$4.P2
- new net P15: IC1.GPB6, Q14.G, U$4.P3
- new net P16: IC1.GPB7, Q15.G, U$4.P4
- new net P2: IC1.GPA1, Q1.G, U$1.P2
- new net P3: IC1.GPA2, Q2.G, U$1.P3
- new net P4: IC1.GPA3, Q3.G, U$1.P4
- new net P5: IC1.GPA4, Q4.G, U$2.P1
- new net P6: IC1.GPA5, Q5.G, U$2.P2
- new net P7: IC1.GPA6, Q6.G, U$2.P3
- new net P8: IC1.GPA7, Q7.G, U$2.P4
- new net P9: IC1.GPB0, Q8.G, U$3.P1
- new net SCL: CON1.SCL, CON2.SCL, IC1.SCL, R20.2
- new net SDA: CON1.SDA, CON2.SDA, IC1.SDA, R19.2
- new net VCC: C2.1, C3.1, C4.+, IC1.!RESET, IC1.VDD, LED18.A, Q0.S, Q1.S, Q10.S, Q11.S, Q12.S, Q13.S, Q14.S, Q15.S, Q2.S, Q3.S, Q4.S, Q5.S, Q6.S, Q7.S, Q8.S, Q9.S, R1.2, R2.2, R3.2, SCL.2, SDA.2, U$1.5V, U$2.5V, U$3.5V, U$4.5V, VR1.OUT
Other:
- note added: "Feedback LEDs"
- note added: "I2C Expander card based on IOX16"
- note added: "John Plocher"
- note removed: "A Template for Eagle Projects"
- note removed: "Your Name"
